File: hardware/industrial-counter-bricklet.kicad_pcb (KiCad board)
At the start: 2 copper layers, 40 x 40 mm, 45 parts, among them J1 DEBUG, P1 CON-SENSOR2, P2 BOOT, P3 CONN_8, U1 XMC1XXX48, U2 TLP2367, U3 TLP2367, U4 TLP2367, U5 TLP2367, U6 DRILL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

Commit message: fix mounting hole
Parts:
- U6, U7, U8, U9: footprint DRILL_NP -> kicad-libraries:DRILL_NP
Changed lines of the file:
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@@
     )
   )
-  (module DRILL_NP (layer Front)
-    (at 100.29952 75.54976)
-    (clearance 0.89916)
-    (fp_text reference U6 (at 0 0) (layer F.SilkS) hide
-      (effects (font (size 0.29972 0.29972) (thickness 0.0762)))
-    )
-    (fp_text value DRILL (at 0 0.50038) (layer F.SilkS) hide
-      (effects (font (size 0.29972 0.29972) (thickness 0.0762)))
-    )
-    (fp_circle (center 0 0) (end 2.19964 -0.20066) (layer F.SilkS) (width 0.381))
-    (fp_circle (center 0 0) (end 1.99898 -0.20066) (layer F.SilkS) (width 0.381))
-    (fp_circle (center 0 0) (end 1.69926 0) (layer F.SilkS) (width 0.381))
-    (fp_circle (center 0 0) (end 1.39954 -0.09906) (layer B.SilkS) (width 0.381))
-    (fp_circle (center 0 0) (end 1.39954 0) (layer F.SilkS) (width 0.381))
-    (fp_circle (center 0 0) (end 1.69926 0) (layer B.SilkS) (width 0.381))
-    (fp_circle (center 0 0) (end 1.89992 0) (layer B.SilkS) (width 0.381))
-    (fp_circle (center 0 0) (end 2.19964 0) (layer B.SilkS) (width 0.381))
-    (pad "" thru_hole circle (at 0 0) (size 2.99974 2.99974) (drill 2.99974) (layers *.Cu *.SilkS *.Mask)
-      (clearance 0.89916))
-  )
   (module Fiducial_Mark (layer Front)
     (at 99.3013 71.54926)
@@
     )
   )
-  (module DRILL_NP (layer Front)
-    (at 100.3 40.55)
-    (fp_text reference U7 (at 0 0) (layer F.SilkS) hide
-      (effects (font (size 0.29972 0.29972) (thickness 0.0762)))
-    )
-    (fp_text value DRILL (at 0 0.50038) (layer F.SilkS) hide
-      (effects (font (size 0.29972 0.29972) (thickness 0.0762)))
-    )
-    (fp_circle (center 0 0) (end 3.2 0) (layer Eco2.User) (width 0.01))
-    (fp_circle (center 0 0) (end 2.19964 -0.20066) (layer F.SilkS) (width 0.381))
-    (fp_circle (center 0 0) (end 1.99898 -0.20066) (layer F.SilkS) (width 0.381))
-    (fp_circle (center 0 0) (end 1.69926 0) (layer F.SilkS) (width 0.381))
-    (fp_circle (center 0 0) (end 1.39954 -0.09906) (layer B.SilkS) (width 0.381))
-    (fp_circle (center 0 0) (end 1.39954 0) (layer F.SilkS) (width 0.381))
-    (fp_circle (center 0 0) (end 1.69926 0) (layer B.SilkS) (width 0.381))
-    (fp_circle (center 0 0) (end 1.89992 0) (layer B.SilkS) (width 0.381))
-    (fp_circle (center 0 0) (end 2.19964 0) (layer B.SilkS) (width 0.381))
-    (pad "" np_thru_hole circle (at 0 0) (size 2.99974 2.99974) (drill 2.99974) (layers *.Cu *.Mask F.SilkS)
-      (clearance 0.89916))
-  )
-  (module DRILL_NP (layer Front)
-    (at 135.3 75.55)
-    (fp_text reference U8 (at 0 0) (layer F.SilkS) hide
-      (effects (font (size 0.29972 0.29972) (thickness 0.0762)))
-    )
-    (fp_text value DRILL (at 0 0.50038) (layer F.SilkS) hide
-      (effects (font (size 0.29972 0.29972) (thickness 0.0762)))
-    )
-    (fp_circle (center 0 0) (end 3.2 0) (layer Eco2.User) (width 0.01))
-    (fp_circle (center 0 0) (end 2.19964 -0.20066) (layer F.SilkS) (width 0.381))
-    (fp_circle (center 0 0) (end 1.99898 -0.20066) (layer F.SilkS) (width 0.381))
-    (fp_circle (center 0 0) (end 1.69926 0) (layer F.SilkS) (width 0.381))
-    (fp_circle (center 0 0) (end 1.39954 -0.09906) (layer B.SilkS) (width 0.381))
-    (fp_circle (center 0 0) (end 1.39954 0) (layer F.SilkS) (width 0.381))
-    (fp_circle (center 0 0) (end 1.69926 0) (layer B.SilkS) (width 0.381))
-    (fp_circle (center 0 0) (end 1.89992 0) (layer B.SilkS) (width 0.381))
-    (fp_circle (center 0 0) (end 2.19964 0) (layer B.SilkS) (width 0.381))
-    (pad "" np_thru_hole circle (at 0 0) (size 2.99974 2.99974) (drill 2.99974) (layers *.Cu *.Mask F.SilkS)
-      (clearance 0.89916))
-  )
-  (module DRILL_NP (layer Front)
-    (at 135.3 40.55)
-    (fp_text reference U9 (at 0 0) (layer F.SilkS) hide
-      (effects (font (size 0.29972 0.29972) (thickness 0.0762)))
-    )
-    (fp_text value DRILL (at 0 0.50038) (layer F.SilkS) hide
-      (effects (font (size 0.29972 0.29972) (thickness 0.0762)))
-    )
-    (fp_circle (center 0 0) (end 3.2 0) (layer Eco2.User) (width 0.01))
-    (fp_circle (center 0 0) (end 2.19964 -0.20066) (layer F.SilkS) (width 0.381))
-    (fp_circle (center 0 0) (end 1.99898 -0.20066) (layer F.SilkS) (width 0.381))
-    (fp_circle (center 0 0) (end 1.69926 0) (layer F.SilkS) (width 0.381))
-    (fp_circle (center 0 0) (end 1.39954 -0.09906) (layer B.SilkS) (width 0.381))
-    (fp_circle (center 0 0) (end 1.39954 0) (layer F.SilkS) (width 0.381))
-    (fp_circle (center 0 0) (end 1.69926 0) (layer B.SilkS) (width 0.381))
-    (fp_circle (center 0 0) (end 1.89992 0) (layer B.SilkS) (width 0.381))
-    (fp_circle (center 0 0) (end 2.19964 0) (layer B.SilkS) (width 0.381))
-    (pad "" np_thru_hole circle (at 0 0) (size 2.99974 2.99974) (drill 2.99974) (layers *.Cu *.Mask F.SilkS)
-      (clearance 0.89916))
-  )
   (module kicad-libraries:CE_5mm (layer Back)
     (at 107.8 58.05 90)
@@
       (xy 1.301301 2.715081) (xy 1.302426 2.714986)) (layer B.SilkS) (width 0.01))
   )
+  (module kicad-libraries:DRILL_NP (layer Front)
+    (at 135.3 40.55)
+    (fp_text reference U9 (at 0 0) (layer F.SilkS) hide
+      (effects (font (size 0.29972 0.29972) (thickness 0.0762)))
+    )
+    (fp_text value DRILL (at 0 0.50038) (layer F.SilkS) hide
+      (effects (font (size 0.29972 0.29972) (thickness 0.0762)))
+    )
+    (fp_circle (center 0 0) (end 3.2 0) (layer Eco2.User) (width 0.01))
+    (fp_circle (center 0 0) (end 2.19964 -0.20066) (layer F.SilkS) (width 0.381))
+    (fp_circle (center 0 0) (end 1.99898 -0.20066) (layer F.SilkS) (width 0.381))
+    (fp_circle (center 0 0) (end 1.69926 0) (layer F.SilkS) (width 0.381))
+    (fp_circle (center 0 0) (end 1.39954 -0.09906) (layer B.SilkS) (width 0.381))
+    (fp_circle (center 0 0) (end 1.39954 0) (layer F.SilkS) (width 0.381))
+    (fp_circle (center 0 0) (end 1.69926 0) (layer B.SilkS) (width 0.381))
+    (fp_circle (center 0 0) (end 1.89992 0) (layer B.SilkS) (width 0.381))
+    (fp_circle (center 0 0) (end 2.19964 0) (layer B.SilkS) (width 0.381))
+    (pad "" np_thru_hole circle (at 0 0) (size 2.99974 2.99974) (drill 2.99974) (layers *.Cu *.Mask F.SilkS)
+      (clearance 0.89916))
+  )
+  (module kicad-libraries:DRILL_NP (layer Front)
+    (at 135.3 75.55)
+    (fp_text reference U8 (at 0 0) (layer F.SilkS) hide
+      (effects (font (size 0.29972 0.29972) (thickness 0.0762)))
+    )
+    (fp_text value DRILL (at 0 0.50038) (layer F.SilkS) hide
+      (effects (font (size 0.29972 0.29972) (thickness 0.0762)))
+    )
+    (fp_circle (center 0 0) (end 3.2 0) (layer Eco2.User) (width 0.01))
+    (fp_circle (center 0 0) (end 2.19964 -0.20066) (layer F.SilkS) (width 0.381))
+    (fp_circle (center 0 0) (end 1.99898 -0.20066) (layer F.SilkS) (width 0.381))
+    (fp_circle (center 0 0) (end 1.69926 0) (layer F.SilkS) (width 0.381))
+    (fp_circle (center 0 0) (end 1.39954 -0.09906) (layer B.SilkS) (width 0.381))
+    (fp_circle (center 0 0) (end 1.39954 0) (layer F.SilkS) (width 0.381))
+    (fp_circle (center 0 0) (end 1.69926 0) (layer B.SilkS) (width 0.381))
+    (fp_circle (center 0 0) (end 1.89992 0) (layer B.SilkS) (width 0.381))
+    (fp_circle (center 0 0) (end 2.19964 0) (layer B.SilkS) (width 0.381))
+    (pad "" np_thru_hole circle (at 0 0) (size 2.99974 2.99974) (drill 2.99974) (layers *.Cu *.Mask F.SilkS)
+      (clearance 0.89916))
+  )
+  (module kicad-libraries:DRILL_NP (layer Front)
+    (at 100.3 40.55)
+    (fp_text reference U7 (at 0 0) (layer F.SilkS) hide
+      (effects (font (size 0.29972 0.29972) (thickness 0.0762)))
+    )
+    (fp_text value DRILL (at 0 0.50038) (layer F.SilkS) hide
+      (effects (font (size 0.29972 0.29972) (thickness 0.0762)))
+    )
+    (fp_circle (center 0 0) (end 3.2 0) (layer Eco2.User) (width 0.01))
+    (fp_circle (center 0 0) (end 2.19964 -0.20066) (layer F.SilkS) (width 0.381))
+    (fp_circle (center 0 0) (end 1.99898 -0.20066) (layer F.SilkS) (width 0.381))
+    (fp_circle (center 0 0) (end 1.69926 0) (layer F.SilkS) (width 0.381))
+    (fp_circle (center 0 0) (end 1.39954 -0.09906) (layer B.SilkS) (width 0.381))
+    (fp_circle (center 0 0) (end 1.39954 0) (layer F.SilkS) (width 0.381))
+    (fp_circle (center 0 0) (end 1.69926 0) (layer B.SilkS) (width 0.381))
+    (fp_circle (center 0 0) (end 1.89992 0) (layer B.SilkS) (width 0.381))
+    (fp_circle (center 0 0) (end 2.19964 0) (layer B.SilkS) (width 0.381))
+    (pad "" np_thru_hole circle (at 0 0) (size 2.99974 2.99974) (drill 2.99974) (layers *.Cu *.Mask F.SilkS)
+      (clearance 0.89916))
+  )
+  (module kicad-libraries:DRILL_NP (layer Front)
+    (at 100.29952 75.54976)
+    (fp_text reference U6 (at 0 0) (layer F.SilkS) hide
+      (effects (font (size 0.29972 0.29972) (thickness 0.0762)))
+    )
+    (fp_text value DRILL (at 0 0.50038) (layer F.SilkS) hide
+      (effects (font (size 0.29972 0.29972) (thickness 0.0762)))
+    )
+    (fp_circle (center 0 0) (end 3.2 0) (layer Eco2.User) (width 0.01))
+    (fp_circle (center 0 0) (end 2.19964 -0.20066) (layer F.SilkS) (width 0.381))
+    (fp_circle (center 0 0) (end 1.99898 -0.20066) (layer F.SilkS) (width 0.381))
+    (fp_circle (center 0 0) (end 1.69926 0) (layer F.SilkS) (width 0.381))
+    (fp_circle (center 0 0) (end 1.39954 -0.09906) (layer B.SilkS) (width 0.381))
+    (fp_circle (center 0 0) (end 1.39954 0) (layer F.SilkS) (width 0.381))
+    (fp_circle (center 0 0) (end 1.69926 0) (layer B.SilkS) (width 0.381))
+    (fp_circle (center 0 0) (end 1.89992 0) (layer B.SilkS) (width 0.381))
+    (fp_circle (center 0 0) (end 2.19964 0) (layer B.SilkS) (width 0.381))
+    (pad "" np_thru_hole circle (at 0 0) (size 2.99974 2.99974) (drill 2.99974) (layers *.Cu *.Mask F.SilkS)
+      (clearance 0.89916))
+  )
   (gr_text 3 (at 131.1 42.7) (layer F.SilkS)
