File: hardware/industrial-counter-bricklet.kicad_pcb (KiCad board)
At the start: 2 copper layers, 40 x 40 mm, 45 parts, among them J1 DEBUG, P1 CON-SENSOR2, P2 BOOT, P3 CONN_8, U1 XMC1XXX48, U2 TLP2367, U3 TLP2367, U4 TLP2367, U5 TLP2367, U6 DRILL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

Commit message: specify processor
Parts:
- U1: value XMC1XXX48 -> XMC1404
Changed lines of the file:
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@@
   (module kicad-libraries:QFN48-EP2 (layer Front)
     (at 105.7 48.45 180)
-    (fp_text reference U1 (at 0 0 180) (layer F.SilkS)
-      (effects (font (size 0.29972 0.29972) (thickness 0.0762)))
+    (fp_text reference U1 (at 0 0 180) (layer F.Fab)
+      (effects (font (size 0.29972 0.29972) (thickness 0.07493)))
     )
-    (fp_text value XMC1XXX48 (at 0 -0.7 180) (layer F.SilkS)
-      (effects (font (size 0.29972 0.29972) (thickness 0.0762)))
+    (fp_text value XMC1404 (at 0 -0.7 180) (layer F.Fab)
+      (effects (font (size 0.29972 0.29972) (thickness 0.07493)))
     )
     (fp_circle (center -2.5 2.6) (end -2.4 2.8) (layer F.Fab) (width 0.05))

Commit message: Add 3d information (final)
Parts:
- U2, U3, U4, U5: footprint SO-5 -> kicad-libraries:SO-5
